File: hardware/smartknob.kicad_sch (KiCad schematic)
At the start: 0 parts

Commit message: feat(hardware): integrate XIAO ESP32-C6 with encoder and display
Add XIAO ESP32-C6 microcontroller to the hardware design and establish
connections to the MT6701 encoder and GC9A01A display. This includes
custom footprints and symbols for the XIAO module, along with complete
schematic integration.

Changes include: - Add XIAO ESP32-C6 custom footprint and symbol
libraries - Add datasheets for ESP32-C6, XIAO ESP32-C6, MT6701 encoder,
and GC9A01A display - Update schematic to wire XIAO ESP32-C6 to encoder
and display - Configure KiCad library tables for custom components
Parts:
- added C1: 10uF, symbol Device:C
- added C2: 0.1uF, symbol Device:C
- added R1, R2, R3, R4, R5: 10k, symbol Device:R
- added TP1, TP2, TP3, TP4, TP5, TP6, TP7, TP8, TP9: TestPoint, symbol Connector:TestPoint
- added U1: XIAO-ESP32-C6, Module:MOUDLE14P-XIAO-DIP-SMD, symbol Seeed_Studio_XIAO_Series:XIAO_ESP32-C6-DIP
Connections:
- new net +3V3: C1.2, C2.2, R1.2, R2.2, R3.2, R4.2, R5.2, TP8.1, U1.12 (3V3)
- new net CLK: TP7.1, U1.9 (GPIO19/D8/SCK)
- new net DISP_CMD: R2.1, TP2.1, U1.2 (GPIO1/A1/D1)
- new net DISP_CS: R1.1, TP1.1, U1.1 (GPIO0/A0/D0)
- new net DISP_RST: R3.1, TP3.1, U1.3 (GPIO2/A2/D2)
- new net ENC_CS: R4.1, TP4.1, U1.4 (GPIO21/D3)
- new net GND: C1.1, C2.1, TP9.1, U1.13 (GND)
- new net MISO: R5.1, TP6.1, U1.10 (GPIO20/D9/MISO)
- new net MOSI: TP5.1, U1.11 (GPIO18/D10/MOSI)
- no-connect marks 0 -> 5
Other:
- note added: "DEBUG"
- note added: "MCU"
