File: hardware/prototypes/driver/driver.kicad_sch (KiCad schematic)
At the start: 46 parts, among them J1 Screw_Terminal_01x02, J2 SPI Connector, J3 Sense Connector, J4 INL Connector, J5 INH Connector, J7 Mode Connector, Q1 AO3401A, U1 DRV8316CRRGFR, U2 PLMR36506RRPET

Commit message: fix: create fake prototype
Parts:
- removed C1, C14, C15, C16, C17, C18, C19, C24, C25, C5, C6, C7, C8: 22uF, symbol Device:C
- removed C10, C11, C9: 30pF, symbol Device:C
- removed C12, C22, C3: 1uF, symbol Device:C
- removed C13, C21, C23, C4: 100nF, symbol Device:C
- removed C2: 47nF, symbol Device:C
- removed C20: 2.2uF, symbol Device:C
- removed H1, H2, H3: MountingHole_Pad, symbol Mechanical:MountingHole_Pad
- removed J1: Screw_Terminal_01x02, symbol Connector:Screw_Terminal_01x02
- removed J2: SPI Connector, symbol Connector:Conn_01x04_Pin
- removed J3: Sense Connector, symbol Connector:Conn_01x04_Pin
- removed J4: INL Connector, symbol Connector:Conn_01x03_Pin
- removed J5: INH Connector, symbol Connector:Conn_01x03_Pin
- removed J7: Mode Connector, symbol Connector:Conn_01x02_Pin
- removed L1: 15uH, symbol Device:L
- removed Q1: AO3401A, Package_TO_SOT_SMD:SOT-23, symbol Transistor_FET:AO3401A
- removed R1: 22, symbol Device:R
- removed R2, R3, R4, R5: 1k, symbol Device:R
- removed R6: 5.1k, symbol Device:R
- removed TP1, TP2: TestPoint, symbol Connector:TestPoint
- removed U2: PLMR36506RRPET, footprints:LMR36506, symbol LMR36506:PLMR36506RRPET
- added J1: POWER_IN, TerminalBlock_Phoenix:TerminalBlock_Phoenix_MKDS-1,5-2_1x02_P5.00mm_Horizontal, symbol Connector_Generic:Conn_01x02
- added U2: ESP32-C6, footprints:ESP32-C6-DevKitC-1_Socket, symbol ESP32-C6:ESP32-C6-DevKitC-1
Connections:
- net GND: now also J1.2 (Pin_2); no longer U1.12 (PGND), U1.15 (PGND), U1.18 (PGND), U1.2 (AGND), U1.26 (AGND), U1.4 (GND_BK), U1.41 (EPAD)
- net +3.3V: no longer names the net of U1.23 (NSLEEP)
- net CLK: no longer names the net of U1.35 (SCLK)
- net CS: no longer names the net of U1.36 (NSCS)
- net DRVOFF: no longer names the net of U1.21 (DRVOFF)
- net INHA: no longer names the net of U1.27 (INHA)
- net INHB: no longer names the net of U1.29 (INHB)
- net INHC: no longer names the net of U1.31 (INHC)
- net INLA: no longer names the net of U1.28 (INLA)
- net INLB: no longer names the net of U1.30 (INLB)
- net INLC: no longer names the net of U1.32 (INLC)
- net NFAULT: no longer names the net of U1.22 (NFAULT)
- net OUTA: no longer names the net of U1.13 (OUTA)
- net OUTA: no longer U1.14 (OUTA)
- net OUTB: no longer names the net of U1.16 (OUTB)
- net OUTB: no longer U1.17 (OUTB)
- net OUTC: no longer names the net of U1.19 (OUTC)
- net OUTC: no longer U1.20 (OUTC)
- net SDI: no longer names the net of U1.34 (SDI)
- net SDO: no longer names the net of U1.33 (SDO)
- removed net VIN: U1.10 (VM), U1.11 (VM), U1.9 (VM)
- net V_BUCK_OUT: no longer names the net of U1.3 (FB_BK)
- new net VM_IN: J1.1 (Pin_1)
- no-connect marks 1 -> 2
