File: hardware/protoypes/driver/driver.kicad_sch (KiCad schematic)
At the start: 0 parts

Commit message: feat: add DRV8316C motor driver schematic and PCB project files
Parts:
- added U1: DRV8316CRRGFR, Footprints:DRV8316CRRGFR, symbol DRV8316CRRGFR:DRV8316CRRGFR
Changed lines of the file:
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@@
 		(company "${COMPANY}")
+	)
+	(symbol
+		(lib_id "DRV8316CRRGFR:DRV8316CRRGFR")
+		(at 62.23 55.88 0)
+		(unit 1)
+		(body_style 1)
+		(exclude_from_sim no)
+		(in_bom yes)
+		(on_board yes)
+		(in_pos_files yes)
+		(dnp no)
+		(fields_autoplaced yes)
+		(property "Reference" "U1"
+			(at 90.17 45.72 0)
+			(show_name no)
+			(do_not_autoplace no)
+			(effects
+				(font
+					(size 1.524 1.524)
+				)
+			)
+		)
+		(property "Value" "DRV8316CRRGFR"
+			(at 90.17 48.26 0)
+			(show_name no)
+			(do_not_autoplace no)
+			(effects
+				(font
+					(size 1.524 1.524)
+				)
+			)
+		)
+		(property "Footprint" "Footprints:DRV8316CRRGFR"
+			(at 62.23 55.88 0)
+			(hide yes)
+			(show_name no)
+			(do_not_autoplace no)
+			(effects
+				(font
+					(size 1.27 1.27)
+					(italic yes)
+				)
+			)
+		)
+		(property "Datasheet" "https://www.ti.com/lit/gpn/drv8316c"
+			(at 62.23 55.88 0)
+			(hide yes)
+			(show_name no)
+			(do_not_autoplace no)
+			(effects
+				(font
+					(size 1.27 1.27)
+					(italic yes)
+				)
+			)
+		)
+		(property "Description" ""
+			(at 62.23 55.88 0)
+			(hide yes)
+			(show_name no)
+			(do_not_autoplace no)
+			(effects
+				(font
+					(size 1.27 1.27)
+				)
+			)
+		)
+		(pin "20"
+		)
+		(pin "19"
+		)
+		(pin "13"
+		)
+		(pin "15"
+		)
+		(pin "22"
+		)
+		(pin "28"
+		)
+		(pin "34"
+		)
+		(pin "33"
+		)
+		(pin "12"
+		)
+		(pin "17"
+		)
+		(pin "18"
+		)
+		(pin "6"
+		)
+		(pin "7"
+		)
+		(pin "14"
+		)
+		(pin "27"
+		)
+		(pin "21"
+		)
+		(pin "26"
+		)
+		(pin "25"
+		)
+		(pin "16"
+		)
+		(pin "5"
+		)
+		(pin "4"
+		)
+		(pin "24"
+		)
+		(pin "23"
+		)
+		(pin "41"
+		)
+		(pin "2"
+		)
+		(pin "3"
+		)
+		(pin "11"
+		)
+		(pin "8"
+		)
+		(pin "9"
+		)
+		(pin "10"
+		)
+		(pin "38"
+		)
+		(pin "40"
+		)
+		(pin "39"
+		)
+		(pin "37"
+		)
+		(pin "36"
+		)
+		(pin "35"
+		)
+		(pin "1"
+		)
+		(pin "29"
+		)
+		(pin "32"
+		)
+		(pin "31"
+		)
+		(pin "30"
+		)
+		(instances
+			(project "driver"
+				(path "/640ae8de-2758-4a23-8a49-1eca08669922"
+					(reference "U1")
+					(unit 1)
+				)
+			)
+		)
 	)
 	(sheet_instances
